Commit message: Created gazebo with obstacle

File: description/robot_core.xacro (robot description, xacro)
@@ -2,4 +2,5 @@
 <robot xmlns:xacro="http://www.ros.org/wiki/xacro"  >
     <xacro:include filename="inertial_macros.xacro" />
+    <xacro:include filename="gazebo_control.xacro" />
         <material name="white">
         <color rgba="1 1 1 1"/>
@@ -39,4 +40,7 @@
     </xacro:inertial_box>
         </link>
+        <gazebo reference="chassis">
+            <material>Gazebo/White</material>
+        </gazebo>
 <!-- LEFT WHEEL -->
 <joint name="left_wheel_joint" type="continuous">
@@ -62,4 +66,7 @@
     </xacro:inertial_cylinder>
 </link>
+<gazebo reference="left_wheel">
+    <material>Gazebo/Blue</material>
+</gazebo>
 <!-- RIGHT WHEEL -->
 <joint name="right_wheel_joint" type="continuous">
@@ -85,4 +92,7 @@
     </xacro:inertial_cylinder>
 </link>
+<gazebo reference="right_wheel">
+    <material>Gazebo/Blue</material>
+</gazebo>
 <!-- CASTER WHEEL -->
 <joint name="caster_wheel_joint" type="fixed">
@@ -107,3 +117,6 @@
     </xacro:inertial_sphere>
 </link>
+<gazebo reference="caster_wheel">
+    <material>Gazebo/Black</material>
+</gazebo>
 </robot>
