Commit message: Created lidar and camera

File: description/robot.urdf.xacro (robot description, xacro)
@@ -2,3 +2,6 @@
 <robot xmlns:xacro="http://www.ros.org/wiki/xacro"  name="robot">
 <xacro:include filename="robot_core.xacro" />
+<xacro:include filename="gazebo_control.xacro" />
+<xacro:include filename="lidar.xacro" />
+<xacro:include filename="camera.xacro" />
 </robot>

File: description/robot_core.xacro (robot description, xacro)
@@ -2,5 +2,4 @@
 <robot xmlns:xacro="http://www.ros.org/wiki/xacro"  >
     <xacro:include filename="inertial_macros.xacro" />
-    <xacro:include filename="gazebo_control.xacro" />
         <material name="white">
         <color rgba="1 1 1 1"/>
@@ -8,4 +7,7 @@
         <material name="orange">
             <color rgba="1 0.3 0.1 1"/>
+        </material>
+        <material name="red">
+            <color rgba="1 0 0 1"/>
         </material>
         <material name="blue">
